File: pcb/NostrZapLamp.kicad_sch (KiCad schematic)
At the start: 4 parts, among them J1 LED, J2 Button, U1 ESP32_DevKit_V1_DOIT

Commit message: PCB tweaks. Update gitignore to exclude kicad locks
Connections:
- net at BZ1.2 (+), U1.14 (GND): now also J1.2 (Pin_2); no longer J1.1 (Pin_1)
- net at U1.13 (IO13): now also J1.1 (Pin_1); no longer J1.2 (Pin_2)
Changed lines of the file:
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@@
     (stroke (width 0) (type default))
   )
-  (wire (pts (xy 138.43 60.96) (xy 138.43 134.62))
+  (wire (pts (xy 160.02 60.96) (xy 132.08 60.96))
     (stroke (width 0) (type default))
   )
-  (wire (pts (xy 160.02 63.5) (xy 127 63.5))
+  (wire (pts (xy 132.08 77.47) (xy 121.92 77.47))
     (stroke (width 0) (type default))
   )
   (wire (pts (xy 146.05 78.74) (xy 160.02 78.74))
+    (stroke (width 0) (type default))
+  )
+  (wire (pts (xy 160.02 63.5) (xy 138.43 63.5))
     (stroke (width 0) (type default))
   )
@@
     (stroke (width 0) (type default))
   )
-  (wire (pts (xy 160.02 60.96) (xy 138.43 60.96))
+  (wire (pts (xy 138.43 63.5) (xy 138.43 134.62))
     (stroke (width 0) (type default))
   )
@@
     (stroke (width 0) (type default))
   )
-  (wire (pts (xy 127 77.47) (xy 121.92 77.47))
-    (stroke (width 0) (type default))
-  )
   (wire (pts (xy 106.68 128.27) (xy 106.68 125.73))
     (stroke (width 0) (type default))
@@
     (stroke (width 0) (type default))
   )
+  (wire (pts (xy 132.08 60.96) (xy 132.08 77.47))
+    (stroke (width 0) (type default))
+  )
   (wire (pts (xy 160.02 93.98) (xy 127 93.98))
     (stroke (width 0) (type default))
   )
-  (wire (pts (xy 127 63.5) (xy 127 77.47))
-    (stroke (width 0) (type default))
-  )
